Commit message: feat(hardware): 新增重力补偿支持，优化关节控制逻辑
- easyarm_hardware 新增 easyarm_dynamics 依赖，通过 URDF/Pinocchio 计算各关节重力力矩并在 write() 中施加

- 新增 ros2_control 参数：urdf_path、enable_gravity_compensation、gravity_compensation_scale

- 新增 parse_bool_parameter() 辅助方法

- command_kp 由 20.0 调整为 10.0；移除阻尼回退模式（allow_position_control）

- 补充 write() 控制流水线中文注释，说明各模块意图

- easyarm_a1_moveit_config xacro 增加 easyarm_urdf_path 参数化 URDF 路径

- AGENTS.md 更新构建与 lint 命令说明

- 新增 docs/ 目录，收录电机通信协议参考文档

注：重力补偿仅在 MotionControl 模式下生效，position_csp 下会有 warning。已在真实硬件上验证，效果符合预期。

File: src/easyarm_a1_moveit_config/config/EasyARM-A1.ros2_control.xacro (robot description, xacro)
@@ -1,5 +1,5 @@
 <?xml version="1.0"?>
 <robot xmlns:xacro="http://www.ros.org/wiki/xacro">
-    <xacro:macro name="EasyARM-A1_ros2_control" params="name initial_positions_file">
+    <xacro:macro name="EasyARM-A1_ros2_control" params="name initial_positions_file urdf_path">
         <xacro:property name="initial_positions" value="${load_yaml(initial_positions_file)['initial_positions']}"/>
         <ros2_control name="${name}" type="system">
@@ -9,4 +9,7 @@
                 <param name="host_can_id">0xFD</param>
                 <param name="use_mock_hardware">false</param>
+                <param name="urdf_path">${urdf_path}</param>
+                <param name="enable_gravity_compensation">true</param>
+                <param name="gravity_compensation_scale">1.0</param>
                 <param name="position_kp">100.0</param>
                 <param name="position_kd">4.0</param>

File: src/easyarm_a1_moveit_config/config/EasyARM-A1.urdf.xacro (robot description, xacro)
@@ -2,8 +2,12 @@
 <robot xmlns:xacro="http://www.ros.org/wiki/xacro" name="EasyARM-A1">
     <xacro:arg name="initial_positions_file" default="initial_positions.yaml" />
+    <xacro:arg name="easyarm_urdf_path" default="$(find easyarm_description)/urdf/easyarm_a1_h0521.urdf" />
     <!-- Import EasyARM-A1 urdf file -->
-    <xacro:include filename="$(find easyarm_description)/urdf/easyarm_a1_h0521.urdf" />
+    <xacro:include filename="$(arg easyarm_urdf_path)" />
     <!-- Import control_xacro -->
     <xacro:include filename="EasyARM-A1.ros2_control.xacro" />
-    <xacro:EasyARM-A1_ros2_control name="EasyArmHardware" initial_positions_file="$(arg initial_positions_file)"/>
+    <xacro:EasyARM-A1_ros2_control
+        name="EasyArmHardware"
+        initial_positions_file="$(arg initial_positions_file)"
+        urdf_path="$(arg easyarm_urdf_path)"/>
 </robot>

Commit message: feat(hardware): 增加硬件调试日志
新增 easyarm_hardware 二进制调试日志、后台落盘线程和离线解析绘图脚本。

demo.launch.py 增加 debug_log_enabled 参数，默认关闭；开启后日志写入 /dev/shm/easyarm_log_YYYYMMDD_HHMMSS.bin。

验证：colcon build --packages-select easyarm_hardware easyarm_a1_moveit_config；用户已完成实机测试。

File: src/easyarm_a1_moveit_config/config/EasyARM-A1.ros2_control.xacro (robot description, xacro)
@@ -1,5 +1,5 @@
 <?xml version="1.0"?>
 <robot xmlns:xacro="http://www.ros.org/wiki/xacro">
-    <xacro:macro name="EasyARM-A1_ros2_control" params="name initial_positions_file urdf_path">
+    <xacro:macro name="EasyARM-A1_ros2_control" params="name initial_positions_file urdf_path debug_log_enabled">
         <xacro:property name="initial_positions" value="${load_yaml(initial_positions_file)['initial_positions']}"/>
         <ros2_control name="${name}" type="system">
@@ -26,9 +26,11 @@
                 <param name="control_mode">motion_control</param>
                 <!-- <param name="control_mode">position_csp</param> -->
+                <param name="debug_log_enabled">${debug_log_enabled}</param>
+                <param name="debug_buffer_seconds">60</param>
             </hardware>
             <joint name="Joint1">
                 <param name="motor_id">0x01</param>
                 <param name="motor_type">RS00</param>
-                <param name="direction">-1.0</param>
+                <param name="direction">1.0</param>
                 <param name="position_offset">0.0</param>
                 <command_interface name="position">

File: src/easyarm_a1_moveit_config/config/EasyARM-A1.urdf.xacro (robot description, xacro)
@@ -3,4 +3,5 @@
     <xacro:arg name="initial_positions_file" default="initial_positions.yaml" />
     <xacro:arg name="easyarm_urdf_path" default="$(find easyarm_description)/urdf/easyarm_a1_h0521.urdf" />
+    <xacro:arg name="debug_log_enabled" default="false" />
     <!-- Import EasyARM-A1 urdf file -->
     <xacro:include filename="$(arg easyarm_urdf_path)" />
@@ -10,4 +11,5 @@
         name="EasyArmHardware"
         initial_positions_file="$(arg initial_positions_file)"
-        urdf_path="$(arg easyarm_urdf_path)"/>
+        urdf_path="$(arg easyarm_urdf_path)"
+        debug_log_enabled="$(arg debug_log_enabled)"/>
 </robot>

File: src/easyarm_description/urdf/easyarm_a1_h0521.urdf (robot description, URDF)
Before this commit: robot EasyARM-A1, 7 links, 6 joints
Joints:
- joint Joint1: axis 0 0 1 -> 0 0 -1

File: src/easyarm_description/urdf/easyarm_a1_h0521_test.urdf (robot description, URDF)
Before this commit: robot EasyARM-A1, 7 links, 6 joints
Joints:
- joint Joint1: origin xyz=0 0 0.0734 rpy=0 0 0 -> xyz=0 0 0.0734 rpy=0 3.1416538 0
- joint Joint2: origin xyz=0 0.073 0 rpy=-1.5708 1.5708 0 -> xyz=0 0.073 0 rpy=-1.5708 -1.5708 0

Commit message: feat(move-task): 更新轨迹记录路径和回放提示
- 将 easyarm_record 默认输出目录改为 data/path_record\n- 优化 easyarm_replay_rviz 缺失文件提示\n- 同步 MoveIt 配置与硬件控制参数调整文档\n\n已运行: colcon build --packages-select easyarm_hardware easyarm_a1_moveit_config easyarm_move_task\n\n涉及硬件控制参数和写周期行为调整，未做真实硬件测试。

File: src/easyarm_a1_moveit_config/config/EasyARM-A1.ros2_control.xacro (robot description, xacro)
@@ -1,5 +1,5 @@
 <?xml version="1.0"?>
 <robot xmlns:xacro="http://www.ros.org/wiki/xacro">
-    <xacro:macro name="EasyARM-A1_ros2_control" params="name initial_positions_file urdf_path debug_log_enabled">
+    <xacro:macro name="EasyARM-A1_ros2_control" params="name initial_positions_file urdf_path debug_enable">
         <xacro:property name="initial_positions" value="${load_yaml(initial_positions_file)['initial_positions']}"/>
         <ros2_control name="${name}" type="system">
@@ -26,5 +26,5 @@
                 <param name="control_mode">motion_control</param>
                 <!-- <param name="control_mode">position_csp</param> -->
-                <param name="debug_log_enabled">${debug_log_enabled}</param>
+                <param name="debug_enable">${debug_enable}</param>
                 <param name="debug_buffer_seconds">60</param>
             </hardware>

File: src/easyarm_a1_moveit_config/config/EasyARM-A1.urdf.xacro (robot description, xacro)
@@ -3,5 +3,5 @@
     <xacro:arg name="initial_positions_file" default="initial_positions.yaml" />
     <xacro:arg name="easyarm_urdf_path" default="$(find easyarm_description)/urdf/easyarm_a1_h0521.urdf" />
-    <xacro:arg name="debug_log_enabled" default="false" />
+    <xacro:arg name="debug_enable" default="false" />
     <!-- Import EasyARM-A1 urdf file -->
     <xacro:include filename="$(arg easyarm_urdf_path)" />
@@ -12,4 +12,4 @@
         initial_positions_file="$(arg initial_positions_file)"
         urdf_path="$(arg easyarm_urdf_path)"
-        debug_log_enabled="$(arg debug_log_enabled)"/>
+        debug_enable="$(arg debug_enable)"/>
 </robot>

Commit message: feat(moveit): 增加仿真硬件启动参数

File: src/easyarm_a1_moveit_config/config/EasyARM-A1.ros2_control.xacro (robot description, xacro)
@@ -1,5 +1,5 @@
 <?xml version="1.0"?>
 <robot xmlns:xacro="http://www.ros.org/wiki/xacro">
-    <xacro:macro name="EasyARM-A1_ros2_control" params="name initial_positions_file urdf_path debug_enable">
+    <xacro:macro name="EasyARM-A1_ros2_control" params="name initial_positions_file urdf_path debug_enable use_mock_hardware">
         <xacro:property name="initial_positions" value="${load_yaml(initial_positions_file)['initial_positions']}"/>
         <ros2_control name="${name}" type="system">
@@ -8,5 +8,5 @@
                 <param name="can_interface">can0</param>
                 <param name="host_can_id">0xFD</param>
-                <param name="use_mock_hardware">false</param>
+                <param name="use_mock_hardware">${use_mock_hardware}</param>
                 <param name="urdf_path">${urdf_path}</param>
                 <param name="enable_gravity_compensation">true</param>

File: src/easyarm_a1_moveit_config/config/EasyARM-A1.urdf.xacro (robot description, xacro)
@@ -4,4 +4,5 @@
     <xacro:arg name="easyarm_urdf_path" default="$(find easyarm_description)/urdf/easyarm_a1_h0521.urdf" />
     <xacro:arg name="debug_enable" default="false" />
+    <xacro:arg name="use_mock_hardware" default="false" />
     <!-- Import EasyARM-A1 urdf file -->
     <xacro:include filename="$(arg easyarm_urdf_path)" />
@@ -12,4 +13,5 @@
         initial_positions_file="$(arg initial_positions_file)"
         urdf_path="$(arg easyarm_urdf_path)"
-        debug_enable="$(arg debug_enable)"/>
+        debug_enable="$(arg debug_enable)"
+        use_mock_hardware="$(arg use_mock_hardware)"/>
 </robot>
