Commit message: feat(moveit): 同步 h0616 硬件配置
将 easyarm_a1_h0616_moveit_config 的 ros2_control、控制器、launch 参数和依赖同步到 0521 硬件配置。

保留 H0616 自碰撞矩阵不变。

已测试。

File: src/easyarm_a1_h0616_moveit_config/config/easyarm_a1.ros2_control.xacro (robot description, xacro)
@@ -1,52 +1,139 @@
 <?xml version="1.0"?>
 <robot xmlns:xacro="http://www.ros.org/wiki/xacro">
-    <xacro:macro name="easyarm_a1_ros2_control" params="name initial_positions_file">
+    <xacro:macro name="easyarm_a1_ros2_control" params="name initial_positions_file urdf_path debug_enable use_mock_hardware">
         <xacro:property name="initial_positions" value="${load_yaml(initial_positions_file)['initial_positions']}"/>
         <ros2_control name="${name}" type="system">
             <hardware>
-                <!-- By default, set up controllers for simulation. This won't work on real hardware -->
-                <plugin>mock_components/GenericSystem</plugin>
+                <plugin>easyarm_hardware/EasyArmHardware</plugin>
+                <param name="can_interface">can0</param>
+                <param name="host_can_id">0xFD</param>
+                <param name="use_mock_hardware">${use_mock_hardware}</param>
+                <param name="urdf_path">${urdf_path}</param>
+                <param name="enable_gravity_compensation">true</param>
+                <param name="hardware_control_mode">position</param>
+                <param name="gravity_compensation_scale">1.0</param>
+                <param name="idle_kd">4.0</param>
+                <param name="drag_gravity_scale">1.0</param>
+                <param name="drag_kd">0.00</param>
+                <param name="control_torque_limit_scale">1.0</param>
+                <param name="position_kp">50.0</param>
+                <param name="position_kd">4.0</param>
+                <param name="velocity_limit">10.0</param>
+                <param name="smoothing_alpha">0.8</param>
+                <param name="max_velocity">2.0</param>
+                <param name="max_acceleration">8.0</param>
+                <param name="control_period">0.005</param>
+                <param name="control_mode">motion_control</param>
+                <!-- <param name="control_mode">position_csp</param> -->
+                <param name="debug_enable">${debug_enable}</param>
+                <param name="debug_buffer_seconds">60</param>
             </hardware>
             <joint name="Joint1">
-                <command_interface name="position"/>
+                <param name="motor_id">0x01</param>
+                <param name="motor_type">RS00</param>
+                <param name="direction">1.0</param>
+                <param name="position_offset">0.0</param>
+                <command_interface name="position">
+                    <param name="min">-3.14</param>
+                    <param name="max">3.14</param>
+                </command_interface>
+                <command_interface name="velocity"/>
+                <command_interface name="effort"/>
                 <state_interface name="position">
                   <param name="initial_value">${initial_positions['Joint1']}</param>
                 </state_interface>
                 <state_interface name="velocity"/>
+                <state_interface name="effort"/>
+                <state_interface name="temperature"/>
             </joint>
             <joint name="Joint2">
-                <command_interface name="position"/>
+                <param name="motor_id">0x02</param>
+                <param name="motor_type">RS00</param>
+                <param name="direction">1.0</param>
+                <param name="position_offset">0.0</param>
+                <command_interface name="position">
+                    <param name="min">-3.14</param>
+                    <param name="max">3.14</param>
+                </command_interface>
+                <command_interface name="velocity"/>
+                <command_interface name="effort"/>
                 <state_interface name="position">
                   <param name="initial_value">${initial_positions['Joint2']}</param>
                 </state_interface>
                 <state_interface name="velocity"/>
+                <state_interface name="effort"/>
+                <state_interface name="temperature"/>
             </joint>
             <joint name="Joint3">
-                <command_interface name="position"/>
+                <param name="motor_id">0x03</param>
+                <param name="motor_type">RS00</param>
+                <param name="direction">1.0</param>
+                <param name="position_offset">0.0</param>
+                <command_interface name="position">
+                    <param name="min">-3.14</param>
+                    <param name="max">3.14</param>
+                </command_interface>
+                <command_interface name="velocity"/>
+                <command_interface name="effort"/>
                 <state_interface name="position">
                   <param name="initial_value">${initial_positions['Joint3']}</param>
                 </state_interface>
                 <state_interface name="velocity"/>
+                <state_interface name="effort"/>
+                <state_interface name="temperature"/>
             </joint>
             <joint name="Joint4">
-                <command_interface name="position"/>
+                <param name="motor_id">0x04</param>
+                <param name="motor_type">RS00</param>
+                <param name="direction">1.0</param>
+                <param name="position_offset">0.0</param>
+                <command_interface name="position">
+                    <param name="min">-3.14</param>
+                    <param name="max">3.14</param>
+                </command_interface>
+                <command_interface name="velocity"/>
+                <command_interface name="effort"/>
                 <state_interface name="position">
                   <param name="initial_value">${initial_positions['Joint4']}</param>
                 </state_interface>
                 <state_interface name="velocity"/>
+                <state_interface name="effort"/>
+                <state_interface name="temperature"/>
             </joint>
             <joint name="Joint5">
-                <command_interface name="position"/>
+                <param name="motor_id">0x05</param>
+                <param name="motor_type">RS00</param>
+                <param name="direction">1.0</param>
+                <param name="position_offset">0.0</param>
+                <command_interface name="position">
+                    <param name="min">-3.14</param>
+                    <param name="max">3.14</param>
+                </command_interface>
+                <command_interface name="velocity"/>
+                <command_interface name="effort"/>
                 <state_interface name="position">
                   <param name="initial_value">${initial_positions['Joint5']}</param>
                 </state_interface>
                 <state_interface name="velocity"/>
+                <state_interface name="effort"/>
+                <state_interface name="temperature"/>
             </joint>
             <joint name="Joint6">
-                <command_interface name="position"/>
+                <param name="motor_id">0x06</param>
+                <param name="motor_type">EL05</param>
+                <param name="direction">1.0</param>
+                <param name="position_offset">0.0</param>
+                <command_interface name="position">
+                    <param name="min">-3.14</param>
+                    <param name="max">3.14</param>
+                </command_interface>
+                <command_interface name="velocity"/>
+                <command_interface name="effort"/>
                 <state_interface name="position">
                   <param name="initial_value">${initial_positions['Joint6']}</param>
                 </state_interface>
                 <state_interface name="velocity"/>
+                <state_interface name="effort"/>
+                <state_interface name="temperature"/>
             </joint>
         </ros2_control>

File: src/easyarm_a1_h0616_moveit_config/config/easyarm_a1.urdf.xacro (robot description, xacro)
@@ -2,8 +2,16 @@
 <robot xmlns:xacro="http://www.ros.org/wiki/xacro" name="easyarm_a1">
     <xacro:arg name="initial_positions_file" default="initial_positions.yaml" />
+    <xacro:arg name="easyarm_urdf_path" default="$(find easyarm_description)/urdf/easyarm_a1_h0616.urdf" />
+    <xacro:arg name="debug_enable" default="false" />
+    <xacro:arg name="use_mock_hardware" default="false" />
     <!-- Import easyarm_a1 urdf file -->
-    <xacro:include filename="$(find easyarm_description)/urdf/easyarm_a1_h0616.urdf" />
+    <xacro:include filename="$(arg easyarm_urdf_path)" />
     <!-- Import control_xacro -->
     <xacro:include filename="easyarm_a1.ros2_control.xacro" />
-    <xacro:easyarm_a1_ros2_control name="FakeSystem" initial_positions_file="$(arg initial_positions_file)"/>
+    <xacro:easyarm_a1_ros2_control
+        name="EasyArmHardware"
+        initial_positions_file="$(arg initial_positions_file)"
+        urdf_path="$(arg easyarm_urdf_path)"
+        debug_enable="$(arg debug_enable)"
+        use_mock_hardware="$(arg use_mock_hardware)"/>
 </robot>

Commit message: feat(description): 新增 H0617 标定模型配置
- 新增 H0617 xacro/config 描述和 h0617_cali 标定参数

- 将 H0616 URDF 替换为标定后的模型并保留旧备份

- 新增质量/质心标定工具和常用脚本 wrapper

- 修复 safe shutdown 对 H0616 MoveIt demo 的进程匹配

File: src/easyarm_a1_h0616_moveit_config/config/easyarm_a1.ros2_control.xacro (robot description, xacro)
@@ -15,5 +15,5 @@
                 <param name="idle_kd">4.0</param>
                 <param name="drag_gravity_scale">1.0</param>
-                <param name="drag_kd">0.00</param>
+                <param name="drag_kd">0.10</param>
                 <param name="control_torque_limit_scale">1.0</param>
                 <param name="position_kp">50.0</param>

File: src/easyarm_description/urdf/easyarm_a1_h0616.urdf (robot description, URDF)
Before this commit: robot ass_easyarm_a1_h0616.SLDASM, 7 links, 6 joints
Links:
- link Link2: mass 0.31461 -> 0.7744593105296842
- link Link3: mass 0.188161905183098 -> 0.5040220986569005
- link Link4: mass 0.14848 -> 0.38512475677337077
- link Link5: mass 0.045369 -> 0.06752108176639557
- link Link6: mass 0.016496 -> 0.019926349172910973
Joints:
- joint Joint1: axis 0 0 1 -> 0.0 0.0 1.0; origin xyz=0 0 0.058 rpy=3.1416 0 0 -> xyz=0.0 0.0 0.058 rpy=3.1416 0.0 0.0
- joint Joint2: axis 0 0 1 -> 0.0 0.0 1.0; origin xyz=0 -0.045 -0.0214 rpy=-1.5708 0 0 -> xyz=0.0 -0.045 -0.0214 rpy=-1.5708 0.0 0.0
- joint Joint3: axis 0 0 -1 -> 0.0 0.0 -1.0; origin xyz=0 0.18 0 rpy=0 0 0 -> xyz=0.0 0.18 0.0 rpy=0.0 0.0 0.0
- joint Joint4: axis 0 0 -1 -> 0.0 0.0 -1.0; origin xyz=0 0.172 0.0176 rpy=3.1416 0 0 -> xyz=0.0 0.172 0.0176 rpy=3.1416 0.0 0.0
- joint Joint5: axis 0 0 -1 -> 0.0 0.0 -1.0; origin xyz=0 -0.0214 0.045 rpy=1.5708 0 0 -> xyz=0.0 -0.0214 0.045 rpy=1.5708 0.0 0.0
- joint Joint6: axis 0 0 -1 -> 0.0 0.0 -1.0; origin xyz=0 0.037 0.0399 rpy=-1.5708 0 0 -> xyz=0.0 0.037 0.0399 rpy=-1.5708 0.0 0.0
