Commit message: feat(motion): 增加预设位姿接口和任务脚本
- 新增 MoveNamedState action 和 ListNamedState service，motion server 可直接执行 SRDF group_state。

- easyarm_app 增加 move_named_state/list_named_state CLI，并新增 easyarm_task1 任务脚本。

- ServoL 增加外部/内部目标调试和 target governor，降低目标跨越导致的速度突变。

- description 增加 flange link，MoveIt Servo 末端改为 flange，并更新 RViz 配置。

测试：colcon build --packages-select easyarm_interfaces easyarm_motion_server easyarm_app easyarm_a1_moveit_config

真机测试：用户已完成。

File: src/easyarm_description/urdf/easyarm_a1_h0617.urdf.xacro (robot description, xacro)
@@ -19,3 +19,9 @@
   <xacro:easyarm_link name="Link6" links="${links}" inertials="${inertials}" />
   <xacro:easyarm_joint name="Joint6" joints="${joints}" />
+  <link name="flange" />
+  <joint name="Link6_to_flange" type="fixed">
+    <origin xyz="0 0 0" rpy="0 0 0" />
+    <parent link="Link6" />
+    <child link="flange" />
+  </joint>
 </robot>

Commit message: feat(control): 接入 TCP 工具坐标系
新增 tool2 可视模型和 tcp 固定坐标系，将 MoveIt Servo 与 motion server 默认末端切换到 tcp。

同时记录上电反馈同步竞态风险，并将前端手柄 ServoL 姿态积分改用 Three.js Quaternion。

File: src/easyarm_description/urdf/easyarm_a1_h0617.urdf.xacro (robot description, xacro)
@@ -25,3 +25,25 @@
     <child link="flange" />
   </joint>
+  <link name="tool2">
+    <visual>
+      <origin xyz="0 0 0" rpy="0 0 0"/>
+      <geometry>
+        <mesh filename="package://easyarm_description/meshes/tools/ASS_Tool_2.stl"/>
+      </geometry>
+      <material name="tool_gray">
+        <color rgba="0.45 0.45 0.45 1.0"/>
+      </material>
+    </visual>
+  </link>
+  <joint name="flange_to_tool2" type="fixed">
+    <origin xyz="0 0 0" rpy="0 0 0"/>
+    <parent link="flange"/>
+    <child link="tool2"/>
+  </joint>
+  <link name="tcp"/>
+  <joint name="flange_to_tcp" type="fixed">
+    <origin xyz="0 0 0.04" rpy="0 0 0"/>
+    <parent link="flange"/>
+    <child link="tcp"/>
+  </joint>
 </robot>
